File: CPDB/CPDB/CPDB.kicad_pcb (KiCad board)
At the start: 2 copper layers, 38 x 38 mm, 24 parts, among them U1 INA219BxDCN, U2 TPS54302DDCR, U3 TPS563240DDCR

Commit message: Schematic completed.
Parts:
- removed R2, R3: 3.3K, Resistor_SMD:R_0805_2012Metric
- added C11: 47uF, Capacitor_SMD:C_0805_2012Metric, F.Cu at (192.6, 97.0)
- added C12: 22uF, Capacitor_SMD:C_0805_2012Metric, F.Cu at (192.6, 100.0)
- added J1: Conn_01x02_Pin, Connector_PinHeader_1.00mm:PinHeader_1x02_P1.00mm_Vertical_SMD_Pin1Left, F.Cu at (187.6, 103.6)
- added J2: Conn_01x04_Pin, Connector_PinHeader_1.00mm:PinHeader_1x04_P1.00mm_Vertical_SMD_Pin1Left, F.Cu at (187.6, 98.5)
- R1: value 1M -> 2m; footprint Resistor_SMD:R_Shunt_Ohmite_LVK12 -> Resistor_SMD:R_2512_6332Metric
- R9: value 9.31k -> 9.3k
- moved C10 75.6 mm to (219.1, 140.5)
- moved C7 75.6 mm to (214.8, 141.3)
- moved C8 75.6 mm to (214.8, 143.8)
- moved L1 73.3 mm to (221.8, 108.2)
- moved C1 52.8 mm to (188.8, 134.7)
- moved C2 52.8 mm to (188.8, 137.2)
- moved C3 52.8 mm to (193.0, 134.9)
- moved C4 52.8 mm to (193.0, 137.9)
- moved C6 52.8 mm to (188.8, 142.2)
- moved L2 52.8 mm to (199.6, 139.9)
- moved R4 52.8 mm to (184.6, 126.5)
- moved R6 52.8 mm to (184.6, 132.4)
- moved R7 52.8 mm to (184.6, 135.4)
- moved R8 52.8 mm to (184.6, 138.3)
- moved R9 52.8 mm to (184.6, 141.3)
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Connections:
- C1 pad 1: Net-(U1-IN+) -> V_IN
- R1 pad 1: Net-(R1-Pad1) -> V_IN
- R1 pad 2: V_IN -> GND
- U1 pad 1: Net-(U1-IN+) -> V_IN
- U1 pad 2: Net-(U1-IN-) -> GND
