File: CPDB/CPDB/CPDB.kicad_sch (KiCad schematic)
At the start: 24 parts, among them U1 INA219BxDCN, U2 TPS54302DDCR, U3 TPS563240DDCR

Commit message: CPDB schematic updated
Parts:
- added J1: Conn_01x02_Pin, symbol Connector:Conn_01x02_Pin
- C1, C2, C5, C6, C7, C8: footprint (none) -> Capacitor_SMD:C_0603_1608Metric
- C10, C3, C4, C9: footprint (none) -> Capacitor_SMD:C_0805_2012Metric
- L1: footprint (none) -> Inductor_SMD:L_Chilisin_BMRF00131350
- L2: footprint (none) -> Inductor_SMD:L_Bourns-SRN8040_8x8.15mm
- R1: value R_Shunt -> 20m; footprint (none) -> Resistor_SMD:R_Shunt_Ohmite_LVK12
- R2, R3, R4, R5, R6, R7, R8, R9: footprint (none) -> Resistor_SMD:R_0805_2012Metric
Connections:
- net GND: now also R1.1, R3.1, J1.2 (Pin_2); no longer R1.3
- net V_IN: now also R1.4, R2.1, J1.1 (Pin_1)
- removed net 26V: R1.2
Other:
- note added: "YENIAY"
- note removed: "footprint = 285mm2 ????"
- title: (none) -> CPDB
- moved on the sheet: C1, C10, C2, C3, C4, C5, C6, C7, C8, C9, L1, L2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

Commit message: Schematic completed.
Parts:
- removed R1: 20m, Resistor_SMD:R_Shunt_Ohmite_LVK12, symbol Device:R_Shunt
- removed R2, R3: 3.3K, Resistor_SMD:R_0805_2012Metric, symbol Device:R
- added C11: 47uF, Capacitor_SMD:C_0805_2012Metric, symbol Device:C_Small
- added C12: 22uF, Capacitor_SMD:C_0805_2012Metric, symbol Device:C_Small
- added J2: Conn_01x04_Pin, Connector_PinHeader_1.00mm:PinHeader_1x04_P1.00mm_Vertical_SMD_Pin1Left, symbol Connector:Conn_01x04_Pin
- added R1: 2m, Resistor_SMD:R_2512_6332Metric, symbol Device:R_Small
- J1: footprint (none) -> Connector_PinHeader_1.00mm:PinHeader_1x02_P1.00mm_Vertical_SMD_Pin1Left
- R9: value 9.31k -> 9.3k
Connections:
- net +5V: now also C12.2, J2.1 (Pin_1)
- net 7V: now also C11.2
- net GND: now also U1.2 (IN-), C11.1, C12.1, J2.4 (Pin_4), R1.2
- net I2C_SCL: now also J2.3 (Pin_3)
- net I2C_SDA: now also J2.2 (Pin_2)
- net V_IN: now also C1.1, U1.1 (IN+), R1.1
Other:
- note added: "I2C PIN"
